Commit message: v2

File: export/ur10.urdf (robot description, URDF)
Before this commit: robot ur10, 7 links, 6 joints
Links:
- removed link base
- removed link joint_size_2
- removed link joint_size_2_2
- removed link joint_size_4
- removed link joint_size_4_2
- removed link lower_arm
- removed link tool_flange
- added link arm, mass 0; collision mesh filename=package://ur10_robot_description/meshes/arm.stl; visual mesh filename=package://ur10_robot_description/meshes/arm.stl
- added link claw, mass 0; collision mesh filename=package://ur10_robot_description/meshes/part_1__4.stl; collision mesh filename=package://ur10_robot_description/meshes/part_1__4.stl
- added link planetary_gearbox, mass 0; collision mesh filename=package://ur10_robot_description/meshes/base.stl; collision mesh filename=package://ur10_robot_description/meshes/bearing_10x19x5.stl
- added link planetary_gearbox_2, mass 0; collision mesh filename=package://ur10_robot_description/meshes/bearing_10x19x5.stl; collision mesh filename=package://ur10_robot_description/meshes/bearing_10x19x5.stl
- added link planetary_gearbox_3, mass 0; collision mesh filename=package://ur10_robot_description/meshes/bearing_10x19x5.stl; collision mesh filename=package://ur10_robot_description/meshes/bearing_10x19x5.stl
- added link wrist_pronation, mass 0; collision mesh filename=package://ur10_robot_description/meshes/part_1__3.stl; collision mesh filename=package://ur10_robot_description/meshes/part_6__2.stl
- added link wrist_rotation, mass 0; collision mesh filename=package://ur10_robot_description/meshes/part_1__3.stl; collision mesh filename=package://ur10_robot_description/meshes/part_2.stl
Joints:
- removed joint Revolute_2
- removed joint Revolute_3
- removed joint Revolute_4
- removed joint Revolute_base
- removed joint elbow
- added joint arm: type revolute, parent arm, child planetary_gearbox_3, origin xyz=0.083341 0.055266 -0 rpy=3.14159 -0 -1.93223, axis 0 0 1, limit lower=-3.141592653589793 upper=3.141592653589793 effort=150 velocity=3.15
- added joint base: type revolute, parent planetary_gearbox, child planetary_gearbox_2, origin xyz=-0 0.00144 0.087 rpy=-3.14159 -0 2.51358, axis 0 0 1, limit lower=-3.141592653589793 upper=3.141592653589793 effort=150 velocity=3.15
- added joint wrist1: type revolute, parent planetary_gearbox_3, child wrist_rotation, origin xyz=-0.034446 -0.083155 -0.051001 rpy=1.5708 -0.750346 2.73662, axis 0 0 1, limit lower=-3.141592653589793 upper=3.141592653589793 effort=150 velocity=3.15
- added joint wrist2: type revolute, parent wrist_pronation, child claw, origin xyz=0 0.0699 0.0264 rpy=-1.5708 -0.528968 -3.14159, axis 0 0 1, limit lower=-3.141592653589793 upper=3.141592653589793 effort=150 velocity=3.15
- added joint wristrotate: type revolute, parent wrist_rotation, child wrist_pronation, origin xyz=-0.0264 -0 -0.0423 rpy=-1.5708 1.11985 -1.5708, axis 0 0 1, limit lower=-3.141592653589793 upper=3.141592653589793 effort=150 velocity=3.15
- joint shoulder: child joint_size_4_2 -> arm; limit lower=-0.26588 upper=1.82851 effort=300 velocity=3.15 -> lower=-3.141592653589793 upper=3.141592653589793 effort=300 velocity=3.15; origin xyz=-0 0.086 -0.09 rpy=-1.5708 -0.257718 -3.14159 -> xyz=-0.051 0 -0.05 rpy=-1.5708 0.062436 -1.5708; parent joint_size_4 -> planetary_gearbox_2

File: ros2_ws/src/ur10_robot_description/urdf/ur10.urdf (robot description, URDF)
Before this commit: robot ur10, 8 links, 7 joints
Links:
- removed link base
- removed link environment
- removed link joint_size_2
- removed link joint_size_2_2
- removed link joint_size_4
- removed link joint_size_4_2
- removed link lower_arm
- removed link tool_flange
- added link arm, mass 0; collision mesh filename=package://ur10_robot_description/meshes/arm.stl; visual mesh filename=package://ur10_robot_description/meshes/arm.stl
- added link claw, mass 0; collision mesh filename=package://ur10_robot_description/meshes/part_1__4.stl; collision mesh filename=package://ur10_robot_description/meshes/part_1__4.stl
- added link planetary_gearbox, mass 0; collision mesh filename=package://ur10_robot_description/meshes/base.stl; collision mesh filename=package://ur10_robot_description/meshes/bearing_10x19x5.stl
- added link planetary_gearbox_2, mass 0; collision mesh filename=package://ur10_robot_description/meshes/bearing_10x19x5.stl; collision mesh filename=package://ur10_robot_description/meshes/bearing_10x19x5.stl
- added link planetary_gearbox_3, mass 0; collision mesh filename=package://ur10_robot_description/meshes/bearing_10x19x5.stl; collision mesh filename=package://ur10_robot_description/meshes/bearing_10x19x5.stl
- added link wrist_pronation, mass 0; collision mesh filename=package://ur10_robot_description/meshes/part_1__3.stl; collision mesh filename=package://ur10_robot_description/meshes/part_6__2.stl
- added link wrist_rotation, mass 0; collision mesh filename=package://ur10_robot_description/meshes/part_1__3.stl; collision mesh filename=package://ur10_robot_description/meshes/part_2.stl
Joints:
- removed joint Revolute_2
- removed joint Revolute_3
- removed joint Revolute_4
- removed joint Revolute_base
- removed joint elbow
- removed joint environment_mount
- added joint arm: type revolute, parent arm, child planetary_gearbox_3, origin xyz=0.083341 0.055266 -0 rpy=3.14159 -0 -1.93223, axis 0 0 1, limit lower=-3.141592653589793 upper=3.141592653589793 effort=150 velocity=3.15
- added joint base: type revolute, parent planetary_gearbox, child planetary_gearbox_2, origin xyz=-0 0.00144 0.087 rpy=-3.14159 -0 2.51358, axis 0 0 1, limit lower=-3.141592653589793 upper=3.141592653589793 effort=150 velocity=3.15
- added joint wrist1: type revolute, parent planetary_gearbox_3, child wrist_rotation, origin xyz=-0.034446 -0.083155 -0.051001 rpy=1.5708 -0.750346 2.73662, axis 0 0 1, limit lower=-3.141592653589793 upper=3.141592653589793 effort=150 velocity=3.15
- added joint wrist2: type revolute, parent wrist_pronation, child claw, origin xyz=0 0.0699 0.0264 rpy=-1.5708 -0.528968 -3.14159, axis 0 0 1, limit lower=-3.141592653589793 upper=3.141592653589793 effort=150 velocity=3.15
- added joint wristrotate: type revolute, parent wrist_rotation, child wrist_pronation, origin xyz=-0.0264 -0 -0.0423 rpy=-1.5708 1.11985 -1.5708, axis 0 0 1, limit lower=-3.141592653589793 upper=3.141592653589793 effort=150 velocity=3.15
- joint shoulder: child joint_size_4_2 -> arm; limit lower=-0.26588 upper=1.82851 effort=300 velocity=3.15 -> lower=-3.141592653589793 upper=3.141592653589793 effort=300 velocity=3.15; origin xyz=-0 0.086 -0.09 rpy=-1.5708 -0.257718 -3.14159 -> xyz=-0.051 0 -0.05 rpy=-1.5708 0.062436 -1.5708; parent joint_size_4 -> planetary_gearbox_2
